Commit message: Made seperate xacro for lidar. Added simulated lidar data in dynabot_lidar.xacro so that we can simulate in gazebo and rviz

File: src/dynabot_description/description/dynabot.urdf.xacro (robot description, xacro)
@@ -2,3 +2,4 @@
 <robot xmlns:xacro="http://www.ros.org/wiki/xacro" name="dynabot">
     <xacro:include filename="dynabot_core.xacro" />
+    <xacro:include filename="dynabot_lidar.xacro" />
 </robot>

File: src/dynabot_description/description/dynabot_core.xacro (robot description, xacro)
@@ -186,28 +186,4 @@
         </xacro:inertial_box>
     </link>
-    <!--LIDAR-->
-    <joint name="laser_joint" type="fixed">
-        <parent link="bottom_frame" />
-        <child link="laser" />
-        <origin xyz="0.73915 0 0.1336" />
-    </joint>
-    <link name="laser">
-        <visual>
-            <origin xyz="-0.039775 0 -0.03715" />
-            <geometry>
-                <box size="0.07955 0.0635 0.1143" />
-            </geometry>
-            <material name="red" />
-        </visual>
-        <collision>
-            <origin xyz="-0.039775 0 -0.03715" />
-            <geometry>
-                <box size="0.07955 0.0635 0.1143"  />
-            </geometry>
-        </collision>
-        <xacro:inertial_box mass="0.13" x="0.07955" y="0.0635" z="0.1143">
-            <origin xyz="-0.039775 0 -0.03715" rpy="0 0 0" />
-        </xacro:inertial_box>
-    </link>
     <!--CAMERA-->
     <joint name="camera_joint" type="fixed">

Commit message: Added support for Ros 2 Control

File: src/dynabot_description/description/dynabot.urdf.xacro (robot description, xacro)
@@ -1,6 +1,229 @@
 <?xml version="1.0"?>
-<robot xmlns:xacro="http://www.ros.org/wiki/xacro" name="dynabot">
-    <xacro:include filename="dynabot_core.xacro" />
-    <!-- <xacro:include filename="dynabot_lidar.xacro" /> -->
-    <xacro:include filename="dynabot_gazebo.xacro" />
+<robot name="dynabot" xmlns:xacro="http://www.ros.org/wiki/xacro">
+    <material name="white">
+        <color rgba="1 1 1 1" />
+    </material>
+    <material name="orange">
+        <color rgba="1 0.3 0.1 1"/>
+    </material>
+    <material name="blue">
+        <color rgba="0.2 0.2 1 1"/>
+    </material>
+    <material name="black">
+        <color rgba="0 0 0 1"/>
+    </material>
+    <material name="red">
+        <color rgba="1 0 0 1"/>
+    </material>
+    <xacro:arg name="is_ignition" default="true" />
+    <!--INCLUDE GAZEBO-->
+    <xacro:include filename="$(find dynabot_description)/description/dynabot_gazebo.xacro" />
+    <!--INCLUDE ROS2 CONTROL-->
+    <xacro:include filename="$(find dynabot_description)/description/dynabot_ros2_control.xacro" />
+    <!--BASE LINK-->
+    <link name="base_link"/>
+    <!--CHASSIS LINK-->
+    <link name="chassis">
+        <!--CHASSIS VISUAL-->
+        <visual>
+            <origin xyz="0.5495 0 0.08135" />
+            <geometry>
+                <box size="1.099 0.6689 0.1627" />
+            </geometry>
+            <material name="white" />
+        </visual>
+        <!--CHASSIS COLLISION-->
+        <collision>
+            <origin xyz="0.5495 0 0.08135" />
+            <geometry>
+                <box size="1.099 0.6689 0.1627" />
+            </geometry>
+        </collision>
+        <!--CHASSIS INERTIA-->
+        <inertial>
+            <origin xyz="0.5495 0 0.08135" rpy="0 0 0" />
+            <mass value="29.58" />
+            <inertia ixx="1.081" ixy="0.0" ixz="0.0"
+                    iyy="2.972" iyz="0.0"
+                    izz="3.972" />
+        </inertial>
+    </link>
+    <!--CHASSIS JOINT-->
+    <joint name="chassis_joint" type="fixed">
+        <parent link="base_link" />
+        <child link="chassis" />
+        <origin xyz="-0.5495 0 0" />
+    </joint>
+    <!--BOTTOM FRAME-->
+    <link name="bottom_frame">
+        <visual>
+            <origin xyz="0.3298 0 0.14925" />
+            <geometry>
+                <box size="0.6596 0.6689 0.2985" />
+            </geometry>
+            <material name="white" />
+        </visual>
+        <collision>
+            <origin xyz="0.3298 0 0.14925" />
+            <geometry>
+                <box size="0.6596 0.6689 0.2985" />
+            </geometry>
+        </collision>
+        <inertial>
+            <origin xyz="0.3298 0 0.14925" rpy="0 0 0" />
+            <mass value="8.22" />
+            <inertia ixx="0.244" ixy="0.0" ixz="0.0"
+                    iyy="0.244" iyz="0.0"
+                    izz="0.244" />
+        </inertial>
+    </link>
+    <!--BOTTOM FRAME JOINT-->
+    <joint name="bottom_frame_joint" type="fixed">
+        <parent link="chassis" />
+        <child link="bottom_frame" />
+        <origin xyz="0.2197 0 0.1627" />
+    </joint>
+    <!--TOP FRAME-->
+    <link name="top_frame">
+        <visual>
+            <origin xyz="0.1651 0 0.0762" />
+            <geometry>
+                <box size="0.3302 0.6689 0.1524" />
+            </geometry>
+            <material name="white" />
+        </visual>
+        <collision>
+            <origin xyz="0.1651 0 0.0762" />
+            <geometry>
+                <box size="0.3302 0.6689 0.1524" />
+            </geometry>
+        </collision>
+        <inertial>
+            <origin xyz="0.1651 0 0.0762" rpy="0 0 0" />
+            <mass value="8.22" />
+            <inertia ixx="0.061" ixy="0.0" ixz="0.0"
+                    iyy="0.061" iyz="0.0"
+                    izz="0.061" />
+        </inertial>
+    </link>
+    <!--TOP FRAME JOINT-->
+    <joint name="top_frame_joint" type="fixed">
+        <parent link="bottom_frame" />
+        <child link="top_frame" />
+        <origin xyz="0 0 0.2985" />
+    </joint>
+    <!--LEFT WHEEL LINK-->
+    <link name="left_wheel">
+        <visual>
+            <origin xyz="0 0 0.0681" />
+            <geometry>
+                <cylinder radius="0.202" length=".1362" />
+            </geometry>
+            <material name="blue" />
+        </visual>
+        <collision>
+            <origin xyz="0 0 0.0681" />
+            <geometry>
+                <cylinder radius="0.202" length=".1362" />
+            </geometry>
+        </collision>
+        <inertial>
+            <origin xyz="0 0 0.0681" rpy="0 0 0" />
+            <mass value="6.41" />
+            <inertia ixx="0.131" ixy="0.0" ixz="0.0"
+                    iyy="0.131" iyz="0.0"
+                    izz="0.261" />
+        </inertial>
+    </link>
+    <!--LEFT WHEEL JOINT-->
+    <joint name="left_wheel_joint" type="continuous">
+        <parent link="base_link"/>
+        <child link="left_wheel"/>
+        <origin xyz="0 0.33445 0" rpy="-1.5708 0 0" />
+        <axis xyz="0 0 1" />
+    </joint>
+    <!--RIGHT WHEEL LINK-->
+    <link name="right_wheel">
+        <visual>
+            <origin xyz="0 0 0.0681" />
+            <geometry>
+                <cylinder radius="0.202" length=".1362" />
+            </geometry>
+            <material name="blue" />
+        </visual>
+        <collision>
+            <origin xyz="0 0 0.0681" />
+            <geometry>
+                <cylinder radius="0.202" length=".1362" />
+            </geometry>
+        </collision>
+        <inertial>
+            <origin xyz="0 0 0.0681" rpy="0 0 0" />
+            <mass value="6.41" />
+            <inertia ixx="0.131" ixy="0.0" ixz="0.0"
+                    iyy="0.131" iyz="0.0"
+                    izz="0.261" />
+        </inertial>
+    </link>
+    <!--RIGHT WHEEL JOINT-->
+    <joint name="right_wheel_joint" type="continuous">
+        <parent link="base_link"/>
+        <child link="right_wheel"/>
+        <origin xyz="0 -0.33445 0" rpy="1.5708 0 0" />
+        <axis xyz="0 0 -1" />
+    </joint>
+    <!--FRONT CASTER WHEEL LINK-->
+    <link name="front_caster_wheel">
+        <visual>
+            <geometry>
+                <sphere radius="0.127" />
+            </geometry>
+            <material name="black" />
+        </visual>
+        <collision>
+            <geometry>
+                <sphere radius="0.127" />
+            </geometry>
+        </collision>
+        <inertial>
+            <origin xyz="0 0 0" rpy="0 0 0" />
+            <mass value="2.27" />
+            <inertia ixx="0.001" ixy="0.0" ixz="0.0"
+                    iyy="0.001" iyz="0.0"
+                    izz="0.001" />
+        </inertial>
+    </link>
+    <!--FRONT CASTER WHEEL JOINT-->
+    <joint name="front_caster_wheel_joint" type="fixed">
+        <parent link="chassis" />
+        <child link="front_caster_wheel" />
+        <origin xyz="1.099 0 -0.075" />
+    </joint>
+    <!--REAR CASTER WHEEL LINK-->
+    <link name="rear_caster_wheel">
+        <visual>
+            <geometry>
+                <sphere radius="0.127" />
+            </geometry>
+            <material name="black" />
+        </visual>
+        <collision>
+            <geometry>
+                <sphere radius="0.127" />
+            </geometry>
+        </collision>
+        <inertial>
+            <origin xyz="0 0 0" rpy="0 0 0" />
+            <mass value="2.27" />
+            <inertia ixx="0.001" ixy="0.0" ixz="0.0"
+                    iyy="0.001" iyz="0.0"
+                    izz="0.001" />
+        </inertial>
+    </link>
+    <!--REAR CASTER WHEEL JOINT-->
+    <joint name="rear_caster_wheel_joint" type="fixed">
+        <parent link="chassis" />
+        <child link="rear_caster_wheel" />
+        <origin xyz="0 0 -0.075" />
+    </joint>
 </robot>

File: src/dynabot_description/description/dynabot_gazebo.xacro (robot description, xacro)
@@ -1,8 +1,9 @@
 <?xml version="1.0"?>
-<robot xmlns:xacro="http://www.ros.org/wiki/xacro">
+<robot name="dynabot" xmlns:xacro="http://www.ros.org/wiki/xacro">
+    <!-- Wheels -->
     <gazebo reference="left_wheel">
-        <mu1>10000000000000 </mu1>
-        <mu2>10000000000000</mu2>
-        <kp>100000000000.0</kp>
+        <mu1>1000000000000000.0</mu1>
+        <mu2>1000000000000000.0</mu2>
+        <kp>1000000000000.0</kp>
         <kd>10.0</kd>
         <minDepth>0.001</minDepth>
@@ -11,7 +12,7 @@
     </gazebo>
     <gazebo reference="right_wheel">
-        <mu1>10000000000000</mu1>
-        <mu2>10000000000000</mu2>
-        <kp>100000000000.0</kp>
+        <mu1>1000000000000000.0</mu1>
+        <mu2>1000000000000000.0</mu2>
+        <kp>1000000000000.0</kp>
         <kd>10.0</kd>
         <minDepth>0.001</minDepth>
@@ -19,24 +20,35 @@
         <fdir1>1 0 0</fdir1>
     </gazebo>
-    <gazebo reference="front_caster_wheel">
-        <mu1>0.01</mu1>
-        <mu2>0.01</mu2>
+    <!-- Caster Wheels -->
+    <gazebo reference="rear_caster_wheel">
+        <mu1>0.1</mu1>
+        <mu2>0.1</mu2>
         <kp>1000000.0</kp>
         <kd>100.0</kd>
         <minDepth>0.001</minDepth>
-        <maxVel>0.1</maxVel>
+        <maxVel>1.0</maxVel>
     </gazebo>
-    <gazebo reference="rear_caster_wheel">
-        <mu1>0.01</mu1>
-        <mu2>0.01</mu2>
+    <gazebo reference="front_caster_wheel">
+        <mu1>0.1</mu1>
+        <mu2>0.1</mu2>
         <kp>1000000.0</kp>
         <kd>100.0</kd>
         <minDepth>0.001</minDepth>
-        <maxVel>0.1</maxVel>
+        <maxVel>1.0</maxVel>
     </gazebo>
+    <!-- ROS 2 Control -->
     <gazebo>
-        <plugin filename="ign_ros2_control-system" name="ign_ros2_control::IgnitionROS2ControlPlugin">
-            <parameters> </parameters>
-        </plugin>
+        <!-- ROS 2 Humble -->
+        <xacro:if value="$(arg is_ignition)">
+            <plugin filename="ign_ros2_control-system" name="ign_ros2_control::IgnitionROS2ControlPlugin">
+                <parameters>$(find dynabot_controller)/config/dynabot_controller.yaml</parameters>
+            </plugin>
+        </xacro:if>
+        <!-- ROS 2 Iron or above -->
+        <xacro:unless value="$(arg is_ignition)">
+            <plugin filename="gz_ros2_control-system" name="gz_ros2_control::GazeboSimROS2ControlPlugin">
+                <parameters>$(find dynabot_controller)/config/dynabot_controller.yaml</parameters>
+            </plugin>
+        </xacro:unless>
     </gazebo>
 </robot>

Commit message: Simulated imu data

File: src/dynabot_description/description/dynabot.urdf.xacro (robot description, xacro)
@@ -227,3 +227,34 @@
         <origin xyz="0 0 -0.075" />
     </joint>
+    <!--IMU-->
+    <link name="imu">
+        <!--IMU INERTIAL-->
+        <inertial>
+            <origin xyz="0 0 0" rpy="0 0 0" />
+            <mass value="0.13" />
+            <inertia ixx="0.0000019" ixy="0.0" ixz="0.0"
+                    iyy="0.0000019" iyz="0.0"
+                    izz="0.0000022" />
+        </inertial>
+        <!--IMU VISUAL-->
+        <visual>
+            <origin xyz="0 0 0" rpy="0 0 0" />
+            <geometry>
+                <box size="0.01 0.01 0.007" />
+            </geometry>
+            <material name="black" />
+        </visual>
+        <!--IMU COLLISION-->
+        <collision>
+            <geometry>
+                <box size="0.01 0.01 0.007" />
+            </geometry>
+        </collision>
+    </link>
+    <!--IMU JOINT-->
+    <joint name="imu_joint" type="fixed">
+        <parent link="base_link" />
+        <child link="imu" />
+        <origin xyz="0.658 0 0.2858" rpy="0 0 0" />
+    </joint>
 </robot>

File: src/dynabot_description/description/dynabot_gazebo.xacro (robot description, xacro)
@@ -44,4 +44,6 @@
                 <parameters>$(find dynabot_controller)/config/dynabot_controller.yaml</parameters>
             </plugin>
+            <plugin filename="ignition-gazebo-imu-system" name="ignition::gazebo::systems::Imu">
+            </plugin>
         </xacro:if>
         <!-- ROS 2 Iron or above -->
@@ -50,5 +52,58 @@
                 <parameters>$(find dynabot_controller)/config/dynabot_controller.yaml</parameters>
             </plugin>
+            <plugin filename="gz_ros2_imu-system" name="gz::sim::systems::Imu">
+            </plugin>
         </xacro:unless>
     </gazebo>
+    <!-- IMU -->
+  <gazebo reference="imu_link">
+    <sensor name="imu" type="imu">
+        <always_on>true</always_on>
+        <update_rate>100</update_rate>
+        <gz_frame_id>imu</gz_frame_id>
+        <topic>imu</topic>
+        <imu>
+          <angular_velocity>
+            <x>
+              <noise type="gaussian">
+                <mean>0.0</mean>
+                <stddev>2e-4</stddev>
+              </noise>
+            </x>
+            <y>
+              <noise type="gaussian">
+                <mean>0.0</mean>
+                <stddev>2e-4</stddev>
+              </noise>
+            </y>
+            <z>
+              <noise type="gaussian">
+                <mean>0.0</mean>
+                <stddev>2e-4</stddev>
+              </noise>
+            </z>
+          </angular_velocity>
+          <linear_acceleration>
+            <x>
+              <noise type="gaussian">
+                <mean>0.0</mean>
+                <stddev>1.7e-2</stddev>
+              </noise>
+            </x>
+            <y>
+              <noise type="gaussian">
+                <mean>0.0</mean>
+                <stddev>1.7e-2</stddev>
+              </noise>
+            </y>
+            <z>
+              <noise type="gaussian">
+                <mean>0.0</mean>
+                <stddev>1.7e-2</stddev>
+              </noise>
+            </z>
+          </linear_acceleration>
+        </imu>
+    </sensor>
+  </gazebo>
 </robot>
